File: pcb/sand_drawing/sand_drawing.sch (KiCad schematic (older format))
At the start: 34 parts, among them J0 12V GND, J1 Stepper1, J2 Stepper2, J3 Opto 1, J4 Opto 2, J5 UART, SW1 EN, SW2 IO0, U2 AMS1117-3.3, U3 ESP32-WROOM-32D

Commit message: Nearly finished PCB layout.
Connections:
- net GND: now also J3.1 (Pin_1), J4.1 (Pin_1)
Changed lines of the file:
@@
 Wire Wire Line
 	3150 1300 3150 1200
+$Comp
+L power:GND #PWR?
+U 1 1 5ED1FCFC
+P 1800 7500
+F 0 "#PWR?" H 1800 7250 50  0001 C CNN
+F 1 "GND" H 1805 7327 50  0000 C CNN
+F 2 "" H 1800 7500 50  0001 C CNN
+F 3 "" H 1800 7500 50  0001 C CNN
+	1    1800 7500
+	1    0    0    -1
+$EndComp
 $EndSCHEMATC
