File: pcb/sand_drawing/sand_drawing.sch (KiCad schematic (older format))
At the start: 34 parts, among them J0 12V GND, J1 Stepper1, J2 Stepper2, J3 Opto 1, J4 Opto 2, J5 UART, SW1 EN, SW2 IO0, U2 AMS1117-3.3, U3 ESP32-WROOM-32D

Commit message: Final tweaks. v1.0 PCB done!
Parts:
- added H1, H2, H3, H4: MountingHole, Mounting_Holes:MountingHole_3.2mm_M3, symbol Mechanical:MountingHole
- added LOGO1: Logo_Open_Hardware_Small, Symbols:OSHW-Logo2_14.6x12mm_SilkScreen, symbol Graphic:Logo_Open_Hardware_Small
- C3: value 10µF/25V -> 100pF/50V; LCSC C15850 -> C1790
- R1: footprint Capacitors_SMD:C_0603 -> Resistors_SMD:R_0603
Connections:
- net GND: now also SW1.2
- net at C3.1, U3.3 (EN): now also R1.2, SW1.1; no longer SW1.2
Other:
- moved on the sheet: R1, SW1
Changed lines of the file:
@@
 L Switch:SW_Push SW1
 U 1 1 5EF3FCE6
-P 3150 1900
-F 0 "SW1" V 3104 2048 50  0000 L CNN
-F 1 "EN" V 3195 2048 50  0000 L CNN
-F 2 "Buttons_Switches_THT:SW_PUSH_6mm" H 3150 2100 50  0001 C CNN
-F 3 "~" H 3150 2100 50  0001 C CNN
-	1    3150 1900
+P 3150 2550
+F 0 "SW1" V 3104 2698 50  0000 L CNN
+F 1 "EN" V 3195 2698 50  0000 L CNN
+F 2 "Buttons_Switches_THT:SW_PUSH_6mm" H 3150 2750 50  0001 C CNN
+F 3 "~" H 3150 2750 50  0001 C CNN
+	1    3150 2550
 	0    1    1    0
 $EndComp
@@
 P 2850 2350
 F 0 "C3" V 2700 2300 50  0000 L CNN
-F 1 "10µF/25V" V 3050 2150 50  0000 L CNN
+F 1 "100pF/50V" V 3050 2150 50  0000 L CNN
 F 2 "Capacitors_SMD:C_0805" H 2888 2200 50  0001 C CNN
 F 3 "~" H 2850 2350 50  0001 C CNN
-F 4 "C15850" H 2850 2350 50  0001 C CNN "LCSC"
+F 4 "C1790" H 2850 2350 50  0001 C CNN "LCSC"
 	1    2850 2350
 	0    1    1    0
@@
 Wire Wire Line
 	3000 2350 3150 2350
-Wire Wire Line
-	3150 2100 3150 2350
 Connection ~ 3150 2350
 Wire Wire Line
@@
 L power:+3.3V #PWR0121
 U 1 1 5EF667AF
-P 3150 1200
-F 0 "#PWR0121" H 3150 1050 50  0001 C CNN
-F 1 "+3.3V" H 3165 1373 50  0000 C CNN
-F 2 "" H 3150 1200 50  0001 C CNN
-F 3 "" H 3150 1200 50  0001 C CNN
-	1    3150 1200
+P 3150 1600
+F 0 "#PWR0121" H 3150 1450 50  0001 C CNN
+F 1 "+3.3V" H 3165 1773 50  0000 C CNN
+F 2 "" H 3150 1600 50  0001 C CNN
+F 3 "" H 3150 1600 50  0001 C CNN
+	1    3150 1600
 	1    0    0    -1
 $EndComp
@@
 L Device:R R1
 U 1 1 5EF8D361
-P 3150 1450
-F 0 "R1" H 3220 1496 50  0000 L CNN
-F 1 "10k" H 3220 1405 50  0000 L CNN
-F 2 "Capacitors_SMD:C_0603" V 3080 1450 50  0001 C CNN
-F 3 "~" H 3150 1450 50  0001 C CNN
-F 4 "C25804" H 3150 1450 50  0001 C CNN "LCSC"
-	1    3150 1450
+P 3150 1850
+F 0 "R1" H 3220 1896 50  0000 L CNN
+F 1 "10k" H 3220 1805 50  0000 L CNN
+F 2 "Resistors_SMD:R_0603" V 3080 1850 50  0001 C CNN
+F 3 "~" H 3150 1850 50  0001 C CNN
+F 4 "C25804" H 3150 1850 50  0001 C CNN "LCSC"
+	1    3150 1850
 	1    0    0    -1
 $EndComp
 Wire Wire Line
 	3150 1700 3150 1600
-Wire Wire Line
-	3150 1300 3150 1200
 $Comp
 L power:GND #PWR0123
@@
 	1    0    0    -1
 $EndComp
+$Comp
+L Mechanical:MountingHole H1
+U 1 1 5ED7D409
+P 5450 6900
+F 0 "H1" H 5550 6946 50  0000 L CNN
+F 1 "MountingHole" H 5550 6855 50  0000 L CNN
+F 2 "Mounting_Holes:MountingHole_3.2mm_M3" H 5450 6900 50  0001 C CNN
+F 3 "~" H 5450 6900 50  0001 C CNN
+	1    5450 6900
+	1    0    0    -1
+$EndComp
+$Comp
+L Mechanical:MountingHole H2
+U 1 1 5ED7E268
+P 5450 6700
+F 0 "H2" H 5550 6746 50  0000 L CNN
+F 1 "MountingHole" H 5550 6655 50  0000 L CNN
+F 2 "Mounting_Holes:MountingHole_3.2mm_M3" H 5450 6700 50  0001 C CNN
+F 3 "~" H 5450 6700 50  0001 C CNN
+	1    5450 6700
+	1    0    0    -1
+$EndComp
+$Comp
+L Mechanical:MountingHole H3
+U 1 1 5ED7E771
+P 5450 6500
+F 0 "H3" H 5550 6546 50  0000 L CNN
+F 1 "MountingHole" H 5550 6455 50  0000 L CNN
+F 2 "Mounting_Holes:MountingHole_3.2mm_M3" H 5450 6500 50  0001 C CNN
+F 3 "~" H 5450 6500 50  0001 C CNN
+	1    5450 6500
+	1    0    0    -1
+$EndComp
+$Comp
+L Mechanical:MountingHole H4
+U 1 1 5ED7EB65
+P 5450 6300
+F 0 "H4" H 5550 6346 50  0000 L CNN
+F 1 "MountingHole" H 5550 6255 50  0000 L CNN
+F 2 "Mounting_Holes:MountingHole_3.2mm_M3" H 5450 6300 50  0001 C CNN
+F 3 "~" H 5450 6300 50  0001 C CNN
+	1    5450 6300
+	1    0    0    -1
+$EndComp
+Wire Wire Line
+	3150 2000 3150 2350
+$Comp
+L power:GND #PWR0124
+U 1 1 5ED90583
+P 3150 2750
+F 0 "#PWR0124" H 3150 2500 50  0001 C CNN
+F 1 "GND" H 3155 2577 50  0000 C CNN
+F 2 "" H 3150 2750 50  0001 C CNN
+F 3 "" H 3150 2750 50  0001 C CNN
+	1    3150 2750
+	1    0    0    -1
+$EndComp
+$Comp
+L Graphic:Logo_Open_Hardware_Small LOGO1
+U 1 1 5ED920AB
+P 5500 1150
+F 0 "LOGO1" H 5500 1425 50  0001 C CNN
+F 1 "Logo_Open_Hardware_Small" H 5500 925 50  0001 C CNN
+F 2 "Symbols:OSHW-Logo2_14.6x12mm_SilkScreen" H 5500 1150 50  0001 C CNN
+F 3 "~" H 5500 1150 50  0001 C CNN
+	1    5500 1150
+	1    0    0    -1
+$EndComp
