File: pcb/sand_drawing/sand_drawing.kicad_sch (KiCad schematic)
At the start: 42 parts, among them J0 12V GND, J1 Stepper1, J2 Stepper2, J3 Opto 1, J4 Opto 2, J5 UART, SW1 EN, SW2 IO0, U1 AP63203WU, U2 ESP32-WROOM-32D

Commit message: Add notes to readme, bump version number in schematic drawing, add PCB changelog.
Parts:
- U2: value ESP32-WROOM-32D -> ESP32-WROOM-32D-N16
Changed lines of the file:
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@@
   (paper "A4")
   (title_block
-    (rev "v1.1")
+    (rev "v1.2")
   )
   (junction (at 255.27 118.11) (diameter 0) (color 0 0 0 0)
@@
       (effects (font (size 1.27 1.27)))
     )
-    (property "Value" "ESP32-WROOM-32D" (at 153.67 63.5 0)
+    (property "Value" "ESP32-WROOM-32D-N16" (at 153.67 63.5 0)
       (effects (font (size 1.27 1.27)))
     )
